Commit message: Rearranged quad_description and added xacro file.

File: quad_description/urdf/quadcopter.urdf (robot description, URDF)
Before this commit: robot Final assem.SLDASM, 5 links, 4 joints
Links:
- added link Lidar, mass 0.0131789241976587; collision mesh filename=package://quad_description/meshes/Lidar.STL; visual mesh filename=package://quad_description/meshes/Lidar.STL
- link Link1: mass 0.0102593008371315 -> 0.0102591079722968
- link Link2: mass 0.0102591079734528 -> 0.0102592136005047
- link Link3: mass 0.0102593008234245 -> 0.0102592495590606
- link Link4: mass 0.0102591079590175 -> 0.0102592157047827
- link base_link: mass 0.705203745013749 -> 0.840254267046389
Joints:
- added joint revolute: type continuous, parent base_link, child Lidar, origin xyz=-0.0189949475112854 0 0.22611927995734 rpy=-3.14159265358979 -5.99575093438171E-17 -1.77504932828959, axis 0 0 -1
